Commit message: Removed ompl dependency + 2d point robot

File: my_planar_robot_model/urdf/my_planar_robot.xacro (robot description, xacro)
@@ -29,5 +29,6 @@
     </collision>
   </link>
-  <joint name="joint1" type="continuous">
+</robot>
+  <!-- <joint name="joint1" type="continuous">
     <origin rpy="0 1.57079632679 0" xyz="0 0 0.1"/>
     <parent link="base_link"/>
@@ -84,5 +85,5 @@
         </geometry>
     </collision>
-  </link>
+  </link> -->
   <!-- ROS Control plugin for Gazebo -->
   <gazebo>
